File: PCB/esp8266-battery/esp8266-battery.kicad_pcb (KiCad board)
At the start: 2 copper layers, 29 x 22 mm, 26 parts, among them J1 program, J2 BME280 modul, J3 2xAA, SW1 boot, SW2 reset, U1 ESP-07

Commit message: Update layout to final version
Parts:
- removed the REF** at (138.4, 96.5)
- added P1: ICT-Point, TestPoint:TestPoint_Pad_D1.0mm, F.Cu at (137.7, 93.5)
- added P2: ICT-Point, TestPoint:TestPoint_Pad_D1.0mm, F.Cu at (135.6, 95.5)
- added P3: ICT-Point, TestPoint:TestPoint_Pad_D1.0mm, F.Cu at (135.6, 93.5)
- added P4: ICT-Point, TestPoint:TestPoint_Pad_D1.0mm, F.Cu at (137.7, 95.5)
- moved J3 7.75 mm to (137.2, 106.7), turned to 270 degrees
- moved R6 7.49 mm to (129.5, 103.1)
- moved C3 6.02 mm to (136.1, 103.9), turned to 180 degrees
- moved C4 5.95 mm to (136.1, 102.1), turned to 180 degrees
- moved R5 2.42 mm to (132.1, 103.1)
- moved R7 1.55 mm to (125.0, 95.0)
- moved R8 1.55 mm to (126.5, 95.0)
- moved R2 0.18 mm to (130.3, 100.6)
- moved R3 0.18 mm to (130.3, 99.1)
- moved R4 0.18 mm to (130.3, 97.5)
- moved REF** 0.13 mm to (125.7, 106.2)
- renumbered J3 to J1, J1 to J2, J2 to J3, R3 to R1, R8 to R2, R1 to R3, R2 to R4, R6 to R5, R7 to R6, R4 to R7, R5 to R8, SW2 to SW1, SW1 to SW2
Routing:
- net /IO0: track 23.3 -> 35.1 mm, vias 3 -> 2
- net /~RST: track 11.6 -> 18.8 mm
- net +3V3: track 58.4 -> 64.2 mm, vias 6 -> 2
- net /I2C-SDA: track 22.5 -> 17.1 mm, vias 1 -> 0
- net /I2C-SCL: track 22.5 -> 20.2 mm, vias 3 -> 0
- net Net-(R8-Pad2): track 5.93 -> 4.06 mm
- net Net-(R7-Pad2): track 7.65 -> 6.38 mm
- net Net-(D1-Pad1): track 8.84 -> 9.89 mm
- net /RXD: track 3.51 -> 2.71 mm
